File: Czujniki/_autosave-projekt.kicad_pcb (KiCad board)
At the start: 2 copper layers, 55.9 x 45.7 mm, 57 parts, among them P1 CONN_01X08, P2 CONN_01X06, P3 CONN_01X05, U1 MCP1700, U10 PCA9306, U12 SHTC1, U14 LM4041, U15 MCP6231, U2 PIC16F1703, U3 MCP16251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

Commit message: Commit message
Parts:
- added R6: 10K, Resistors_SMD:R_0603, F.Cu at (214.8, 123.4)
- added R7: 4,7K, Resistors_SMD:R_0603, F.Cu at (209.4, 123.4)
- added R8: 4,7K, Resistors_SMD:R_0603, F.Cu at (207.6, 123.4)
- added T1: Si2323DS, Footprinty:SOT23, F.Cu at (223.3, 122.7)
- added T2: FDV303N, Footprinty:SOT23, F.Cu at (165.0, 124.3)
- added T3: FDV303N, Footprinty:SOT23, F.Cu at (161.3, 124.3)
- moved R5 46.5 mm to (211.2, 123.4), turned to 270 degrees
- moved P2 37.1 mm to (217.5, 111.2), turned to 270 degrees
- moved R2 27.9 mm to (220.7, 122.7), turned to 90 degrees
- moved R1 2.45 mm to (213.0, 123.4), turned to 270 degrees
- moved P3 1.02 mm to (201.3, 111.0)
Connections:
- P2 pad 6: +5V -> Net-(P2-Pad6)
- R2 pad 1: +5V -> Net-(P2-Pad6)
- U2 pad 2: SCL -> SCL5
- U2 pad 3: SDA -> SDA5
- U2 pad 6: (no net) -> CONTROL
Routing:
- net Net-(R6-Pad2): track 0.00 -> 18.0 mm
- net Net-(C3-Pad1): track 0.00 -> 12.9 mm
- net Net-(P2-Pad3): track 0.00 -> 12.6 mm, vias 0 -> 2
- net Net-(P2-Pad6): track 0.00 -> 7.74 mm
- net DUSTOUT: track 0.00 -> 3.65 mm
- net CONTROL: track 0.00 -> 3.54 mm
- net +5V: track 3.10 -> 0.00 mm
- net RESETSIG: track 16.7 -> 19.2 mm
- net SDA5: track 0.00 -> 2.28 mm
- net SCL5: track 0.00 -> 2.28 mm
- net SDA: track 62.7 -> 61.8 mm, vias 3 -> 2
- net SCL: track 63.9 -> 63.0 mm, vias 3 -> 2
- net TRIG: track 2.14 -> 2.99 mm
