File: Czujniki/projekt.sch (KiCad schematic (older format))
At the start: 136 parts, among them P1 CONN_01X02, P2 CONN_01X02, P3 CONN_01X05, P4 CONN_01X02, P5 CONN_01X04, P6 USB_OTG, SW1 SW_PUSH_SMALL, SW2 SW_PUSH_SMALL, T1 Si2323DS, T10 Si2323DS, T11 Si2323DS, T12 2N7002, T13 Si2323DS, T14 Si2323DS, T15 2N7002, T16 Si2323DS, T17 NTD25P03L, T18 2N7002, T2 2N7002, T3 2N7002, T4 NTD25P03L, T5 2N7002, T6 NTD25P03L, T7 NTD25P03L, T8 2N7002, T9 NTD25P03L, U1 MCP73831, U10 PCA9306, U11 24XX1025, U12 SHTC1, U13 HF-LPT100-10, U14 LM4041, U15 MCP6231, U2 dsPIC33EP256MU806, U3 1117, U4 1117, U5 1117, U6 MCP3201, U7 DS1338, U8 MCP6L1, U9 MCP6L1, Y1 Crystal, Y2 ZTCS

Commit message: Working on sensor board
Parts:
- removed C1: 100N, Capacitors_SMD:C_0603_HandSoldering, symbol C_Small
- removed C10, C11, C12, C28, C36, C42, C6, C7, C8: 10U, SMD_Packages:SMD-1206_Pol, symbol CP
- removed C13, C18, C20, C21, C24, C25, C30, C35, C38, C39, C4, C40, C41, C5, C9: 100N, Capacitors_SMD:C_0603_HandSoldering, symbol C
- removed C16: 10U, Capacitors_Tantalum_SMD:TantalC_SizeX_EIA-7343, symbol CP
- removed C2, C3: 4,7u, Footprinty:TantalC_SizeA_EIA-3216_HandSoldering, symbol CP
- removed C23: 100U, SMD_Packages:SMD-1206_Pol, symbol CP
- removed D1, D2: BAS70H, Diodes_SMD:SOD-123, symbol D_Schottky_Small
- removed D3, D4: LL5817, Diodes_SMD:Diode-MELF_Handsoldering, symbol D_Schottky_Small
- removed D5: LED, LEDs:LED-1206, symbol LED
- removed L1: 1n, Resistors_SMD:R_0603, symbol L_Small
- removed P1, P2: CONN_01X02, Pin_Headers:Pin_Header_Straight_1x02, symbol CONN_01X02
- removed P3: CONN_01X05, Socket_Strips:Socket_Strip_Straight_1x05, symbol CONN_01X05
- removed P4: CONN_01X02, Socket_Strips:Socket_Strip_Straight_1x02, symbol CONN_01X02
- removed P5: CONN_01X04, Socket_Strips:Socket_Strip_Straight_1x04, symbol CONN_01X04
- removed P6: USB_OTG, Connect:USB_Mini-B, symbol USB_OTG
- removed R1: 4.7K, Resistors_SMD:R_0603, symbol R
- removed R10, R8: 4,7k, Resistors_SMD:R_0603, symbol R
- removed R11, R12, R15, R16, R17, R19, R23, R3, R32, R34, R35, R36, R4, R5, R9: 100K, Resistors_SMD:R_0603, symbol R
- removed R13, R14: 1M, Resistors_SMD:R_0603, symbol R
- removed R2: 100, Resistors_SMD:R_0603, symbol R
- removed R37, R7: 10K, Resistors_SMD:R_0603, symbol R
- removed R6: 470K, Resistors_SMD:R_0603, symbol R
- removed SW1, SW2: SW_PUSH_SMALL, Footprinty:TACT_SW_ONE_PAIR, symbol SW_PUSH_SMALL
- removed T1, T10, T11: Si2323DS, Footprinty:SOT23, symbol Si2323DS
- removed T12, T15, T18, T2, T3, T5, T8: 2N7002, Footprinty:2N7002-SOT23, symbol 2N7002
- removed T17, T4, T6, T7, T9: NTD25P03L, SMD_Packages:DPAK-3_GDS, symbol NTD25P03L
- removed U1: MCP73831, Housings_SOT-23_SOT-143_TSOT-6:SOT-23-5, symbol MCP73831
- removed U11: 24XX1025, SMD_Packages:SOIC-8-N, symbol 24XX1025
- removed U13: HF-LPT100-10, Footprinty:HF-LPT100-10, symbol HF-LPT100-10
- removed U2: dsPIC33EP256MU806, Housings_QFP:TQFP-64_10x10mm_Pitch0.5mm, symbol dsPIC33EP256MU806
- removed U3, U4, U5: 1117, Footprinty:SOT-223-1117, symbol 1117
- removed Y2: ZTCS, Footprinty:ZTTCS, symbol ZTCS
- added P1: CONN_01X12, Footprinty:DS1065-02-1-12S8BS, symbol CONN_01X12
Connections:
- net labels added: MAIN_VOL
- net labels removed: ?, AVDD, CHARGE_ENABLE, CHARGE_POWER, CHARGE_SIGNAL, CHARGE_STAT, COMM_ENABLE, DM, DP, GNDA, MA0, MA1, MAINTAIN, MEM_ENABLE, MWP, Moduł, OSC1, OSC2, PCLK, PDATA, Pamięć, RESET, RL, RST, SW, TERMINATE, UARTRX, UARTTX, Układ, VBATTERY, VBAT_ADC, VBAT_CONN, VBUS, VINPUT, VON, VPROGSUP, VUSB_BUS, WPWM1, WPWM2, WPWM3, Wi-Fi, mikroprocesora, zasilania, Ładowarka
- wire segments 476 -> 169
- no-connect marks 23 -> 9

Commit message: Simplifiying all
Parts:
- removed C32: 10U, SMD_Packages:SMD-1206_Pol, symbol CP
- removed R24, R33: 100K, Resistors_SMD:R_0603, symbol R
- removed R30: 220K, Resistors_SMD:R_0603, symbol R
- removed T13, T14, T16: Si2323DS, Footprinty:SOT23, symbol Si2323DS
- added C1, C2: 1U, Capacitors_SMD:C_0805_HandSoldering, symbol C_Small
- added U1: MCP1700, Footprinty:SOT23-mcp1700, symbol MCP1700
Connections:
- net labels removed: VDD2
- wire segments 169 -> 158
- no-connect marks 9 -> 8

Commit message: Simplier version - first fixes
Parts:
- removed P1: CONN_01X12, Footprinty:DS1065-02-1-12S8BS, symbol CONN_01X12
- added P1: CONN_01X08, symbol CONN_01X08
Connections:
- net labels added: +3.3V
- net labels removed: CLOCK_ENABLE, CONV_ENABLE, HUM_ENABLE, PRESS_ENABLE, SOUND_ENABLE
- wire segments 158 -> 155
- no-connect marks 8 -> 6
Changed lines of the file:
@@
-$EndComp
-$Comp
-L PWR_FLAG #FLG027
-U 1 1 559E6DFF
-P 8750 10250
-F 0 "#FLG027" H 8750 10345 50  0001 C CNN
-F 1 "PWR_FLAG" H 8750 10430 50  0000 C CNN
-F 2 "" H 8750 10250 60  0000 C CNN
-F 3 "" H 8750 10250 60  0000 C CNN
-	1    8750 10250
-	-1   0    0    1
 $EndComp
 $Comp
@@
 $EndComp
 $Comp
-L GND #PWR028
+L GND #PWR027
 U 1 1 559DA0C7
 P 8450 8400
-F 0 "#PWR028" H 8450 8150 50  0001 C CNN
+F 0 "#PWR027" H 8450 8150 50  0001 C CNN
 F 1 "GND" H 8450 8250 50  0000 C CNN
 F 2 "" H 8450 8400 60  0000 C CNN
@@
 $EndComp
 $Comp
-L GND #PWR029
+L GND #PWR028
 U 1 1 559DCBA3
 P 9800 8350
-F 0 "#PWR029" H 9800 8100 50  0001 C CNN
+F 0 "#PWR028" H 9800 8100 50  0001 C CNN
 F 1 "GND" H 9800 8200 50  0000 C CNN
 F 2 "" H 9800 8350 60  0000 C CNN
@@
 $EndComp
 $Comp
-L GND #PWR030
+L GND #PWR029
 U 1 1 559E9E70
 P 7450 9100
-F 0 "#PWR030" H 7450 8850 50  0001 C CNN
+F 0 "#PWR029" H 7450 8850 50  0001 C CNN
 F 1 "GND" H 7450 8950 50  0000 C CNN
 F 2 "" H 7450 9100 60  0000 C CNN
@@
 $EndComp
 $Comp
-L GND #PWR041
+L GND #PWR030
 U 1 1 559E6A22
 P 7300 6400
-F 0 "#PWR041" H 7300 6150 50  0001 C CNN
+F 0 "#PWR030" H 7300 6150 50  0001 C CNN
 F 1 "GND" H 7300 6250 50  0000 C CNN
 F 2 "" H 7300 6400 60  0000 C CNN
@@
 $EndComp
 $Comp
-L GND #PWR042
+L GND #PWR031
 U 1 1 559EB1FD
 P 7300 6000
-F 0 "#PWR042" H 7300 5750 50  0001 C CNN
+F 0 "#PWR031" H 7300 5750 50  0001 C CNN
 F 1 "GND" H 7300 5850 50  0000 C CNN
 F 2 "" H 7300 6000 60  0000 C CNN
@@
 $EndComp
 $Comp
-L GND #PWR043
+L GND #PWR032
 U 1 1 559EE130
 P 7900 6000
-F 0 "#PWR043" H 7900 5750 50  0001 C CNN
+F 0 "#PWR032" H 7900 5750 50  0001 C CNN
 F 1 "GND" H 7900 5850 50  0000 C CNN
 F 2 "" H 7900 6000 60  0000 C CNN
@@
 	8250 10150 8850 10150
 Wire Wire Line
-	8750 9950 8750 10250
-Wire Wire Line
 	8850 10150 8850 10100
 Wire Wire Line
@@
 	7850 9050 7850 9150
 $Comp
-L GND #PWR044
+L GND #PWR033
 U 1 1 559F20DC
 P 7850 9150
-F 0 "#PWR044" H 7850 8900 50  0001 C CNN
+F 0 "#PWR033" H 7850 8900 50  0001 C CNN
 F 1 "GND" H 7850 9000 50  0000 C CNN
 F 2 "" H 7850 9150 60  0000 C CNN
@@
 	7850 8650 7950 8650
 Connection ~ 7850 8800
-$Comp
-L CONN_01X12 P1
-U 1 1 55AE548B
-P 11850 1850
-F 0 "P1" H 11850 2500 50  0000 C CNN
-F 1 "CONN_01X12" V 11950 1850 50  0000 C CNN
-F 2 "Footprinty:DS1065-02-1-12S8BS" H 11850 1850 60  0001 C CNN
-F 3 "" H 11850 1850 60  0000 C CNN
-	1    11850 1850
-	1    0    0    -1
-$EndComp
-Text GLabel 11600 1300 0    39   Input ~ 0
-SOUND_ENABLE
-Wire Wire Line
-	11600 1300 11650 1300
-Text GLabel 11600 1400 0    39   Input ~ 0
-CONV_ENABLE
-Wire Wire Line
-	11600 1400 11650 1400
-Text GLabel 11600 1500 0    39   Input ~ 0
+Text GLabel 11600 1700 0    39   Input ~ 0
 CLOCK
-Wire Wire Line
-	11600 1500 11650 1500
-Text GLabel 11600 1600 0    39   Input ~ 0
+Text GLabel 11600 1800 0    39   Input ~ 0
 ADCDATA
-Wire Wire Line
-	11600 1600 11650 1600
-Text GLabel 11600 1700 0    39   Input ~ 0
+Text GLabel 11600 1900 0    39   Input ~ 0
 SUSPEND
 Wire Wire Line
 	11600 1700 11650 1700
-Text GLabel 11600 1800 0    39   Input ~ 0
-HUM_ENABLE
 Wire Wire Line
 	11600 1800 11650 1800
-Text GLabel 11600 1900 0    39   Input ~ 0
-PRESS_ENABLE
 Wire Wire Line
 	11600 1900 11650 1900
+Wire Wire Line
+	11600 2000 11650 2000
 Text GLabel 11600 2000 0    39   Input ~ 0
-CLOCK_ENABLE
-Wire Wire Line
-	11600 2000 11650 2000
+SDA
+Wire Wire Line
+	11600 2100 11650 2100
 Text GLabel 11600 2100 0    39   Input ~ 0
-SDA
-Wire Wire Line
-	11600 2100 11650 2100
+SCL
 Text GLabel 11600 2200 0    39   Input ~ 0
-SCL
-Text GLabel 11600 2300 0    39   Input ~ 0
 MAIN_VOL
 $Comp
-L GND #PWR045
+L GND #PWR034
 U 1 1 55AE6E1E
 P 11600 2450
-F 0 "#PWR045" H 11600 2200 50  0001 C CNN
+F 0 "#PWR034" H 11600 2200 50  0001 C CNN
 F 1 "GND" H 11600 2300 50  0000 C CNN
 F 2 "" H 11600 2450 60  0000 C CNN
@@
 	11600 2400 11600 2450
 Wire Wire Line
-	11650 2300 11600 2300
-Wire Wire Line
-	11600 2200 11650 2200
-NoConn ~ 11650 1300
-NoConn ~ 11650 1800
-$Comp
-L PWR_FLAG #FLG048
+	10900 2300 11650 2300
+$Comp
+L PWR_FLAG #FLG035
 U 1 1 55AE93F7
 P 13850 4100
-F 0 "#FLG048" H 13850 4195 50  0001 C CNN
+F 0 "#FLG035" H 13850 4195 50  0001 C CNN
 F 1 "PWR_FLAG" H 13850 4280 50  0000 C CNN
 F 2 "" H 13850 4100 60  0000 C CNN
@@
 $EndComp
 $Comp
-L +1V8 #PWR049
+L +1V8 #PWR036
 U 1 1 55AE94C5
 P 13850 4050
-F 0 "#PWR049" H 13850 3900 50  0001 C CNN
+F 0 "#PWR036" H 13850 3900 50  0001 C CNN
 F 1 "+1V8" H 13850 4190 50  0000 C CNN
 F 2 "" H 13850 4050 60  0000 C CNN
@@
 	13850 4050 13850 4100
 $Comp
-L GND #PWR050
+L GND #PWR037
 U 1 1 55AE9690
 P 11200 5100
-F 0 "#PWR050" H 11200 4850 50  0001 C CNN
+F 0 "#PWR037" H 11200 4850 50  0001 C CNN
 F 1 "GND" H 11200 4950 50  0000 C CNN
 F 2 "" H 11200 5100 60  0000 C CNN
@@
 $EndComp
 $Comp
-L PWR_FLAG #FLG051
+L PWR_FLAG #FLG038
 U 1 1 55AE9702
 P 11200 5050
-F 0 "#FLG051" H 11200 5145 50  0001 C CNN
+F 0 "#FLG038" H 11200 5145 50  0001 C CNN
 F 1 "PWR_FLAG" H 11200 5230 50  0000 C CNN
 F 2 "" H 11200 5050 60  0000 C CNN
@@
 Wire Wire Line
 	11200 5050 11200 5100
-$Comp
-L VDD #PWR052
-U 1 1 55AE9902
-P 9950 3950
-F 0 "#PWR052" H 9950 3800 50  0001 C CNN
-F 1 "VDD" H 9950 4100 50  0000 C CNN
-F 2 "" H 9950 3950 60  0000 C CNN
-F 3 "" H 9950 3950 60  0000 C CNN
-	1    9950 3950
-	1    0    0    -1
-$EndComp
-$Comp
-L PWR_FLAG #FLG053
-U 1 1 55AE9A58
-P 9950 4000
-F 0 "#FLG053" H 9950 4095 50  0001 C CNN
-F 1 "PWR_FLAG" H 9950 4180 50  0000 C CNN
-F 2 "" H 9950 4000 60  0000 C CNN
-F 3 "" H 9950 4000 60  0000 C CNN
-	1    9950 4000
-	-1   0    0    1
-$EndComp
-Wire Wire Line
-	9950 4000 9950 3950
 $Comp
 L MCP1700 U1
@@
 	8750 4550 8750 4600
 $Comp
-L GND #PWR054
+L GND #PWR039
 U 1 1 55AE3407
 P 8750 4600
-F 0 "#PWR054" H 8750 4350 50  0001 C CNN
+F 0 "#PWR039" H 8750 4350 50  0001 C CNN
 F 1 "GND" H 8750 4450 50  0000 C CNN
 F 2 "" H 8750 4600 60  0000 C CNN
@@
 $EndComp
 $Comp
-L GND #PWR055
+L GND #PWR040
 U 1 1 55AE34AF
 P 8300 4600
-F 0 "#PWR055" H 8300 4350 50  0001 C CNN
+F 0 "#PWR040" H 8300 4350 50  0001 C CNN
 F 1 "GND" H 8300 4450 50  0000 C CNN
 F 2 "" H 8300 4600 60  0000 C CNN
@@
 $EndComp
 $Comp
-L GND #PWR056
+L GND #PWR041
 U 1 1 55AE3623
 P 9200 4600
-F 0 "#PWR056" H 9200 4350 50  0001 C CNN
+F 0 "#PWR041" H 9200 4350 50  0001 C CNN
 F 1 "GND" H 9200 4450 50  0000 C CNN
 F 2 "" H 9200 4600 60  0000 C CNN
@@
 Connection ~ 8300 4250
 $Comp
-L +1V8 #PWR057
+L +1V8 #PWR042
 U 1 1 55AE4712
 P 9200 4200
-F 0 "#PWR057" H 9200 4050 50  0001 C CNN
+F 0 "#PWR042" H 9200 4050 50  0001 C CNN
 F 1 "+1V8" H 9200 4340 50  0000 C CNN
 F 2 "" H 9200 4200 60  0000 C CNN
@@
 Connection ~ 9200 4250
 $Comp
-L VDD #PWR?
+L VDD #PWR043
 U 1 1 55AE639E
 P 10500 7950
-F 0 "#PWR?" H 10500 7800 50  0001 C CNN
+F 0 "#PWR043" H 10500 7800 50  0001 C CNN
 F 1 "VDD" H 10500 8100 50  0000 C CNN
 F 2 "" H 10500 7950 60  0000 C CNN
@@
 $EndComp
 $Comp
-L VDD #PWR?
+L VDD #PWR044
 U 1 1 55AE6443
 P 10150 7950
-F 0 "#PWR?" H 10150 7800 50  0001 C CNN
+F 0 "#PWR044" H 10150 7800 50  0001 C CNN
 F 1 "VDD" H 10150 8100 50  0000 C CNN
 F 2 "" H 10150 7950 60  0000 C CNN
@@
 $EndComp
 $Comp
-L VDD #PWR?
+L VDD #PWR045
 U 1 1 55AE64E1
 P 9800 7950
-F 0 "#PWR?" H 9800 7800 50  0001 C CNN
+F 0 "#PWR045" H 9800 7800 50  0001 C CNN
 F 1 "VDD" H 9800 8100 50  0000 C CNN
 F 2 "" H 9800 7950 60  0000 C CNN
@@
 $EndComp
 $Comp
-L VDD #PWR?
+L VDD #PWR046
 U 1 1 55AE657F
 P 9450 7950
-F 0 "#PWR?" H 9450 7800 50  0001 C CNN
+F 0 "#PWR046" H 9450 7800 50  0001 C CNN
 F 1 "VDD" H 9450 8100 50  0000 C CNN
 F 2 "" H 9450 7950 60  0000 C CNN
@@
 $EndComp
 $Comp
-L VDD #PWR?
+L VDD #PWR047
 U 1 1 55AE6B18
 P 8900 8750
-F 0 "#PWR?" H 8900 8600 50  0001 C CNN
+F 0 "#PWR047" H 8900 8600 50  0001 C CNN
 F 1 "VDD" H 8900 8900 50  0000 C CNN
 F 2 "" H 8900 8750 60  0000 C CNN
@@
 $EndComp
 $Comp
-L VDD #PWR?
+L VDD #PWR048
 U 1 1 55AE6C7B
 P 8450 7900
-F 0 "#PWR?" H 8450 7750 50  0001 C CNN
+F 0 "#PWR048" H 8450 7750 50  0001 C CNN
 F 1 "VDD" H 8450 8050 50  0000 C CNN
 F 2 "" H 8450 7900 60  0000 C CNN
@@
 $EndComp
 $Comp
-L VDD #PWR?
+L VDD #PWR049
 U 1 1 55AE6D4B
 P 7450 7850
-F 0 "#PWR?" H 7450 7700 50  0001 C CNN
+F 0 "#PWR049" H 7450 7700 50  0001 C CNN
 F 1 "VDD" H 7450 8000 50  0000 C CNN
 F 2 "" H 7450 7850 60  0000 C CNN
@@
 $EndComp
 $Comp
-L VDD #PWR?
+L VDD #PWR050
 U 1 1 55AE745A
 P 9250 6400
-F 0 "#PWR?" H 9250 6250 50  0001 C CNN
+F 0 "#PWR050" H 9250 6250 50  0001 C CNN
 F 1 "VDD" H 9250 6550 50  0000 C CNN
 F 2 "" H 9250 6400 60  0000 C CNN
@@
 	9250 6450 9250 6400
 $Comp
-L VDD #PWR?
+L VDD #PWR051
 U 1 1 55AE7951
 P 10150 6300
-F 0 "#PWR?" H 10150 6150 50  0001 C CNN
+F 0 "#PWR051" H 10150 6150 50  0001 C CNN
 F 1 "VDD" H 10150 6450 50  0000 C CNN
 F 2 "" H 10150 6300 60  0000 C CNN
@@
 $EndComp
 $Comp
-L VDD #PWR?
+L VDD #PWR052
 U 1 1 55AE80C1
 P 7600 5900
-F 0 "#PWR?" H 7600 5750 50  0001 C CNN
+F 0 "#PWR052" H 7600 5750 50  0001 C CNN
 F 1 "VDD" H 7600 6050 50  0000 C CNN
 F 2 "" H 7600 5900 60  0000 C CNN
@@
 Wire Wire Line
 	12300 6600 12300 6550
+$Comp
+L +3.3V #PWR053
+U 1 1 55AE4376
+P 11200 2250
+F 0 "#PWR053" H 11200 2100 50  0001 C CNN
+F 1 "+3.3V" H 11200 2390 50  0000 C CNN
+F 2 "" H 11200 2250 60  0000 C CNN
+F 3 "" H 11200 2250 60  0000 C CNN
+	1    11200 2250
+	1    0    0    -1
+$EndComp
+Wire Wire Line
+	8750 9950 8750 10150
+$Comp
+L PWR_FLAG #FLG054
+U 1 1 55AE48DD
+P 10900 2250
+F 0 "#FLG054" H 10900 2345 50  0001 C CNN
+F 1 "PWR_FLAG" H 10900 2430 50  0000 C CNN
+F 2 "" H 10900 2250 60  0000 C CNN
+F 3 "" H 10900 2250 60  0000 C CNN
+	1    10900 2250
+	1    0    0    -1
+$EndComp
+Wire Wire Line
+	10900 2250 10900 2300
+$Comp
+L CONN_01X08 P1
+U 1 1 55AE4F37
+P 11850 2050
+F 0 "P1" H 11850 2500 50  0000 C CNN
+F 1 "CONN_01X08" V 11950 2050 50  0000 C CNN
+F 2 "" H 11850 2050 60  0000 C CNN
+F 3 "" H 11850 2050 60  0000 C CNN
+	1    11850 2050
+	1    0    0    -1
+$EndComp
+Wire Wire Line
+	11200 2250 11200 2300
+Connection ~ 11200 2300
+Wire Wire Line
+	11600 2200 11650 2200
 $EndSCHEMATC

Commit message: DC/DC converter to linear converter change
Parts:
- added C?: 10U, symbol CP
- P1: footprint (none) -> Footprinty:DS1065-02-1X8S8BS
Connections:
- net labels added: VDD2
- net labels removed: +3.3V
- wire segments 155 -> 157
Changed lines of the file:
@@
 L GND #PWR01
 U 1 1 5594935A
-P 12400 6750
-F 0 "#PWR01" H 12400 6500 50  0001 C CNN
-F 1 "GND" H 12400 6600 50  0000 C CNN
-F 2 "" H 12400 6750 60  0000 C CNN
-F 3 "" H 12400 6750 60  0000 C CNN
-	1    12400 6750
-	1    0    0    -1
-$EndComp
-$Comp
-L VDD #PWR02
-U 1 1 55949AF6
-P 12300 6550
-F 0 "#PWR02" H 12300 6400 50  0001 C CNN
-F 1 "VDD" H 12300 6700 50  0000 C CNN
-F 2 "" H 12300 6550 60  0000 C CNN
-F 3 "" H 12300 6550 60  0000 C CNN
-	1    12300 6550
+P 12400 7000
+F 0 "#PWR01" H 12400 6750 50  0001 C CNN
+F 1 "GND" H 12400 6850 50  0000 C CNN
+F 2 "" H 12400 7000 60  0000 C CNN
+F 3 "" H 12400 7000 60  0000 C CNN
+	1    12400 7000
 	1    0    0    -1
 $EndComp
@@
 	1    9700 4700
 	-1   0    0    1
-$EndComp
-$Comp
-L VDD #PWR03
-U 1 1 5594E054
-P 9800 4450
-F 0 "#PWR03" H 9800 4300 50  0001 C CNN
-F 1 "VDD" H 9800 4600 50  0000 C CNN
-F 2 "" H 9800 4450 60  0000 C CNN
-F 3 "" H 9800 4450 60  0000 C CNN
-	1    9800 4450
-	1    0    0    -1
 $EndComp
 $Comp
@@
 $EndComp
 $Comp
-L VDD #PWR011
-U 1 1 5595287E
-P 11600 4150
-F 0 "#PWR011" H 11600 4000 50  0001 C CNN
-F 1 "VDD" H 11600 4300 50  0000 C CNN
-F 2 "" H 11600 4150 60  0000 C CNN
-F 3 "" H 11600 4150 60  0000 C CNN
-	1    11600 4150
-	1    0    0    -1
-$EndComp
-$Comp
 L ELECTRET E1
 U 1 1 5595DA45
@@
 	10750 4550 10750 4700
 Wire Wire Line
-	12300 6600 12750 6600
+	12000 6600 12750 6600
 Wire Wire Line
 	12400 6700 12750 6700
 Wire Wire Line
-	12400 6700 12400 6750
+	12400 6700 12400 7000
 Wire Wire Line
 	12700 6800 12750 6800
@@
 $EndComp
 Wire Wire Line
-	12300 6600 12300 6550
-$Comp
-L +3.3V #PWR053
-U 1 1 55AE4376
-P 11200 2250
-F 0 "#PWR053" H 11200 2100 50  0001 C CNN
-F 1 "+3.3V" H 11200 2390 50  0000 C CNN
-F 2 "" H 11200 2250 60  0000 C CNN
-F 3 "" H 11200 2250 60  0000 C CNN
-	1    11200 2250
-	1    0    0    -1
-$EndComp
-Wire Wire Line
 	8750 9950 8750 10150
 $Comp
@@
 F 0 "P1" H 11850 2500 50  0000 C CNN
 F 1 "CONN_01X08" V 11950 2050 50  0000 C CNN
-F 2 "" H 11850 2050 60  0000 C CNN
+F 2 "Footprinty:DS1065-02-1X8S8BS" H 11850 2050 60  0001 C CNN
 F 3 "" H 11850 2050 60  0000 C CNN
 	1    11850 2050
@@
 Wire Wire Line
 	11600 2200 11650 2200
+$Comp
+L CP C?
+U 1 1 55AF6446
+P 12000 6800
+F 0 "C?" H 12025 6900 50  0000 L CNN
+F 1 "10U" H 12025 6700 50  0000 L CNN
+F 2 "" H 12038 6650 30  0000 C CNN
+F 3 "" H 12000 6800 60  0000 C CNN
+	1    12000 6800
+	1    0    0    -1
+$EndComp
+Wire Wire Line
+	12000 6600 12000 6650
+Wire Wire Line
+	12000 6950 12000 7000
+$Comp
+L GND #PWR?
+U 1 1 55AF69F3
+P 12000 7000
+F 0 "#PWR?" H 12000 6750 50  0001 C CNN
+F 1 "GND" H 12000 6850 50  0000 C CNN
+F 2 "" H 12000 7000 60  0000 C CNN
+F 3 "" H 12000 7000 60  0000 C CNN
+	1    12000 7000
+	1    0    0    -1
+$EndComp
+$Comp
+L VDD2 #PWR?
+U 1 1 55AFDFBE
+P 11200 2250
+F 0 "#PWR?" H 11200 2100 50  0001 C CNN
+F 1 "VDD2" H 11200 2400 50  0000 C CNN
+F 2 "" H 11200 2250 60  0000 C CNN
+F 3 "" H 11200 2250 60  0000 C CNN
+	1    11200 2250
+	1    0    0    -1
+$EndComp
+$Comp
+L VDD2 #PWR?
+U 1 1 55AFE0AC
+P 11600 4150
+F 0 "#PWR?" H 11600 4000 50  0001 C CNN
+F 1 "VDD2" H 11600 4300 50  0000 C CNN
+F 2 "" H 11600 4150 60  0000 C CNN
+F 3 "" H 11600 4150 60  0000 C CNN
+	1    11600 4150
+	1    0    0    -1
+$EndComp
+$Comp
+L VDD2 #PWR?
+U 1 1 55AFE87F
+P 9800 4450
+F 0 "#PWR?" H 9800 4300 50  0001 C CNN
+F 1 "VDD2" H 9800 4600 50  0000 C CNN
+F 2 "" H 9800 4450 60  0000 C CNN
+F 3 "" H 9800 4450 60  0000 C CNN
+	1    9800 4450
+	1    0    0    -1
+$EndComp
+$Comp
+L VDD2 #PWR?
+U 1 1 55AFE90E
+P 12250 6550
+F 0 "#PWR?" H 12250 6400 50  0001 C CNN
+F 1 "VDD2" H 12250 6700 50  0000 C CNN
+F 2 "" H 12250 6550 60  0000 C CNN
+F 3 "" H 12250 6550 60  0000 C CNN
+	1    12250 6550
+	1    0    0    -1
+$EndComp
+Wire Wire Line
+	12250 6550 12250 6600
+Connection ~ 12250 6600
 $EndSCHEMATC
