File: Czujniki/_saved_projekt.sch (KiCad schematic (older format))
At the start: 79 parts, among them P1 CONN_01X08, P2 CONN_01X06, P3 CONN_01X05, T1 Si2323DS, T2 FDV303N, T3 FDV303N, T4 Si2323DS, T5 Si2323DS, T6 Si2323DS, T7 Si2323DS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

Commit message: Sensor added in board.
Parts:
- C10, C9: footprint (none) -> Capacitors_SMD:C_0805_HandSoldering
- DET1, DET2: footprint (none) -> Footprinty:MQ-sensor
- R10, R11, R12, R9: footprint (none) -> Resistors_SMD:R_0603
- T4, T5, T6, T7: footprint (none) -> Footprinty:SOT23
- U5: footprint (none) -> Footprinty:SOT23-mcp1700
Changed lines of the file:
@@
 F 0 "DET2" H 5050 8800 60  0000 C CNN
 F 1 "MQ-Sensor" V 4750 8350 60  0000 C CNN
-F 2 "" H 4900 8650 60  0000 C CNN
+F 2 "Footprinty:MQ-sensor" H 4900 8650 60  0001 C CNN
 F 3 "" H 4900 8650 60  0000 C CNN
 	1    4900 8650
@@
 F 0 "R11" V 5230 8850 50  0000 C CNN
 F 1 "R" V 5150 8850 50  0000 C CNN
-F 2 "" V 5080 8850 30  0000 C CNN
+F 2 "Resistors_SMD:R_0603" V 5080 8850 30  0001 C CNN
 F 3 "" H 5150 8850 30  0000 C CNN
 	1    5150 8850
@@
 F 0 "U5" H 1950 5950 60  0000 C CNN
 F 1 "MCP1702" H 1850 6200 60  0000 C CNN
-F 2 "" H 1850 6050 60  0000 C CNN
+F 2 "Footprinty:SOT23-mcp1700" H 1850 6050 60  0001 C CNN
 F 3 "" H 1850 6050 60  0000 C CNN
 	1    1850 6100
@@
 F 0 "T7" H 4750 8350 39  0000 C CNN
 F 1 "Si2323DS" V 4950 8200 39  0000 C CNN
-F 2 "" H 4900 8200 39  0000 C CNN
+F 2 "Footprinty:SOT23" H 4900 8200 39  0001 C CNN
 F 3 "" H 4900 8200 39  0000 C CNN
 	1    4900 8200
@@
 F 0 "R12" H 5330 8220 50  0000 L CNN
 F 1 "100K" H 5330 8160 50  0000 L CNN
-F 2 "" H 5300 8200 60  0000 C CNN
+F 2 "Resistors_SMD:R_0603" H 5300 8200 60  0001 C CNN
 F 3 "" H 5300 8200 60  0000 C CNN
 	1    5300 8200
@@
 F 0 "T6" H 4350 8350 39  0000 C CNN
 F 1 "Si2323DS" V 4550 8200 39  0000 C CNN
-F 2 "" H 4500 8200 39  0000 C CNN
+F 2 "Footprinty:SOT23" H 4500 8200 39  0001 C CNN
 F 3 "" H 4500 8200 39  0000 C CNN
 	1    4500 8200
@@
 F 0 "C10" H 2260 6320 50  0000 L CNN
 F 1 "1U" H 2260 6170 50  0000 L CNN
-F 2 "" H 2250 6250 60  0000 C CNN
+F 2 "Capacitors_SMD:C_0805_HandSoldering" H 2250 6250 60  0001 C CNN
 F 3 "" H 2250 6250 60  0000 C CNN
 	1    2250 6250
@@
 F 0 "C9" H 1460 6320 50  0000 L CNN
 F 1 "1U" H 1460 6170 50  0000 L CNN
-F 2 "" H 1450 6250 60  0000 C CNN
+F 2 "Capacitors_SMD:C_0805_HandSoldering" H 1450 6250 60  0001 C CNN
 F 3 "" H 1450 6250 60  0000 C CNN
 	1    1450 6250
@@
 F 0 "DET1" H 3250 8800 60  0000 C CNN
 F 1 "MQ-Sensor" V 2950 8350 60  0000 C CNN
-F 2 "" H 3100 8650 60  0000 C CNN
+F 2 "Footprinty:MQ-sensor" H 3100 8650 60  0001 C CNN
 F 3 "" H 3100 8650 60  0000 C CNN
 	1    3100 8650
@@
 F 0 "R9" V 3430 8850 50  0000 C CNN
 F 1 "4,7K" V 3350 8850 50  0000 C CNN
-F 2 "" V 3280 8850 30  0000 C CNN
+F 2 "Resistors_SMD:R_0603" V 3280 8850 30  0001 C CNN
 F 3 "" H 3350 8850 30  0000 C CNN
 	1    3350 8850
@@
 F 0 "T5" H 2950 8350 39  0000 C CNN
 F 1 "Si2323DS" V 3150 8200 39  0000 C CNN
-F 2 "" H 3100 8200 39  0000 C CNN
+F 2 "Footprinty:SOT23" H 3100 8200 39  0001 C CNN
 F 3 "" H 3100 8200 39  0000 C CNN
 	1    3100 8200
@@
 F 0 "R10" H 3530 8220 50  0000 L CNN
 F 1 "100K" H 3530 8160 50  0000 L CNN
-F 2 "" H 3500 8200 60  0000 C CNN
+F 2 "Resistors_SMD:R_0603" H 3500 8200 60  0001 C CNN
 F 3 "" H 3500 8200 60  0000 C CNN
 	1    3500 8200
@@
 F 0 "T4" H 2550 8350 39  0000 C CNN
 F 1 "Si2323DS" V 2750 8200 39  0000 C CNN
-F 2 "" H 2700 8200 39  0000 C CNN
+F 2 "Footprinty:SOT23" H 2700 8200 39  0001 C CNN
 F 3 "" H 2700 8200 39  0000 C CNN
 	1    2700 8200
@@
 	4150 1450 4200 1450
 $Comp
-L PWR_FLAG #FLG?
+L PWR_FLAG #FLG089
 U 1 1 55B37391
 P 2450 6050
-F 0 "#FLG?" H 2450 6145 50  0001 C CNN
+F 0 "#FLG089" H 2450 6145 50  0001 C CNN
 F 1 "PWR_FLAG" H 2450 6230 50  0000 C CNN
 F 2 "" H 2450 6050 60  0000 C CNN
