File: Sterownik/projekt.sch (KiCad schematic (older format))
At the start: 57 parts, among them P1 CONN_01X08, P3 CONN_01X05, P4 CONN_01X02, P5 CONN_01X02, P6 USB_OTG, P8 CONN_01X02, SW1 SW_PUSH_SMALL, T10 Si2323DS, T12 2N7002, T18 2N7002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

Commit message: Changed switch placement (from main to sensor board)
Parts:
- removed SW1: SW_PUSH_SMALL, Footprinty:TACT_SW_ONE_PAIR, symbol SW_PUSH_SMALL
Connections:
- net GND: now also U3.4 (GND)
- net TERMINATE: now also P1.2 (P2), U2.64 (AN28/PWM3L/PMD4/RP84/RE4); no longer U2.42 (RTCC/DMLN/RPI72/RD8)
- net VDD: no longer P1.2 (P2)
Other:
- moved on the sheet: R6, T4
